File: stm32f103c8t6.kicad_pcb (KiCad board)
At the start: 2 copper layers, 23.8 x 32.5 mm, 33 parts, among them IC1 AS5600-ASOT, J1 USB4105GFA, J2 SWD_Debugger, J4 DUMMY_PINS, U1 STM32F103C8T6, U2 AMS1117-3.3, Y1 Crystal

Commit message: Add files via upload
Parts:
- C11, C12: value 10p -> 22p; moved to F.Cu
- R2: moved to F.Cu
- moved C3 24.6 mm to (158.1, 78.7), turned to 180 degrees
- moved R7 22.8 mm to (138.8, 91.3)
- moved C2 22.5 mm to (158.1, 77.0), turned to 180 degrees
- moved C8 21.6 mm to (147.1, 71.1), turned to -90 degrees
- moved R2 19.9 mm to (153.4, 90.9), turned to 0 degrees
- moved C15 19.6 mm to (151.1, 83.1), turned to -90 degrees
- moved D1 18.8 mm to (138.7, 89.3)
- moved C13 16.9 mm to (143.2, 71.2)
- moved R6 16.9 mm to (144.9, 71.2), turned to 90 degrees
- moved C12 16.5 mm to (157.7, 72.7), turned to 180 degrees
- moved 120R1 16.3 mm to (148.9, 70.8), turned to 90 degrees
- moved C7 16.3 mm to (152.2, 71.1)
- moved C6 16.3 mm to (150.5, 71.1)
- moved C11 16.0 mm to (157.6, 74.3), turned to 0 degrees
- moved C9 13.4 mm to (145.6, 89.5)
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Routing:
- net GND: track 0.00 -> 58.3 mm, vias 0 -> 12
- net /HSE_OUT: track 41.0 -> 23.4 mm, vias 2 -> 0
- net /BOOT0: track 6.42 -> 22.8 mm, vias 1 -> 2
- net +3.3V: track 78.3 -> 90.6 mm, vias 2 -> 3
- net Net-(D1-A): track 9.50 -> 16.5 mm
- net /SWCLK: track 8.83 -> 15.5 mm
- net Net-(120R1-Pad2): track 8.00 -> 1.95 mm
- net /HSE_IN: track 22.6 -> 16.7 mm, vias 1 -> 0
- net /PB6: track 16.2 -> 11.1 mm
- net /PA0: track 7.35 -> 10.9 mm, vias 1 -> 0
- net /SWDIO: track 13.1 -> 16.2 mm
- net VBUS: track 41.9 -> 39.2 mm, vias 2 -> 4
- net Net-(J1-CC2): track 5.25 -> 3.84 mm
- net Net-(D1-K): track 3.30 -> 2.01 mm
- net /NRST: track 16.3 -> 17.5 mm, vias 0 -> 1
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
Commit message: Add files via upload
final pcb before mounting holes
Routing:
- net /USB_D+: track 0.00 -> 42.8 mm, vias 0 -> 2
- net GND: track 58.3 -> 100.3 mm, vias 12 -> 16
- net /USB_D-: track 0.00 -> 41.3 mm, vias 0 -> 2
- net VBUS: track 39.2 -> 40.8 mm
- net /PB7: track 13.9 -> 15.5 mm
- net +3.3VA: track 19.9 -> 21.0 mm
- net +3.3V: track 90.6 -> 91.5 mm
- net /BOOT0: track 22.8 -> 23.7 mm

Commit message: Add files via upload
final pcb with mounting holes before DFM check
Parts:
- added H1: MountingHole, MountingHole:MountingHole_2.1mm, F.Cu at (134.4, 58.1)
- added H2: MountingHole, MountingHole:MountingHole_2.1mm, F.Cu at (162.1, 58.1)
- added H3: MountingHole, MountingHole:MountingHole_2.1mm, F.Cu at (134.6, 94.4)
- added H4: MountingHole, MountingHole:MountingHole_2.1mm, F.Cu at (162.4, 94.4)
- 120R1: footprint ferrite_bead:BEADC0603X33N -> Inductor_SMD:L_0603_1608Metric_Pad1.05x0.95mm_HandSolder
- moved J1 1.25 mm to (148.6, 62.5)
- moved R3 0.10 mm to (148.8, 83.1)
Routing:
- net GND: track 100.3 -> 106.0 mm
- net VBUS: track 40.8 -> 43.3 mm
- net Net-(J1-CC1): track 3.96 -> 6.24 mm
- net Net-(J1-CC2): track 3.84 -> 6.11 mm
- net /USB_D+: track 42.8 -> 44.4 mm
- net /USB_D-: track 41.3 -> 42.9 mm
Other:
- board size 23.8 x 32.5 mm -> 32.8 x 41.4 mm
