File: stm32f103c8t6.kicad_sch (KiCad schematic)
At the start: 33 parts, among them IC1 AS5600-ASOT, J1 USB4105GFA, J2 SWD_Debugger, J4 DUMMY_PINS, U1 STM32F103C8T6, U2 AMS1117-3.3, Y1 Crystal

Commit message: Add files via upload
Parts:
- C11, C12: value 10p -> 22p
Changed lines of the file:
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@@
 			)
 		)
-		(property "Value" "10p"
+		(property "Value" "22p"
 			(at 31.75 97.7899 0)
 			(effects
@@
 			)
 		)
-		(property "Value" "10p"
+		(property "Value" "22p"
 			(at 52.07 97.7899 0)
 			(effects

Commit message: Add files via upload
final pcb with mounting holes before DFM check
Parts:
- added H1, H2, H3, H4: MountingHole, MountingHole:MountingHole_2.1mm, symbol Mechanical:MountingHole
Other:
- note added: "MOUNTING HOLES"
